Commit message: Adjusted robot model and made robot wheel macro

File: description/robot_core.xacro (robot description, xacro)
@@ -2,4 +2,5 @@
 <robot xmlns:xacro="http://www.ros.org/wiki/xacro">
 <xacro:include filename="inertial_macros.xacro"/>
+<xacro:include filename="robot_macros.xacro"/>
 <material name="white">
     <color rgba="1 1 1 1"/>
@@ -30,5 +31,5 @@
       <geometry>
         <!-- <mesh filename="package://urdf_omni_drive/description/meshes/frame.STL" scale="0.001 0.001 0.001"/> -->
-        <box size="0.7 0.3 0.15"/>
+        <box size="0.75 0.33 0.12"/>
       </geometry>
       <material name="white"/>
@@ -38,8 +39,8 @@
         <geometry>
           <!-- <mesh filename="package://urdf_omni_drive/description/meshes/frame.STL" scale="0.001 0.001 0.001"/> -->
-          <box size="0.7 0.3 0.15"/>
+          <box size="0.75 0.33 0.12"/>
         </geometry>
       </collision>
-      <xacro:inertial_box mass="5" x="0.7" y="0.3" z="0.15">
+      <xacro:inertial_box mass="5" x="0.75" y="0.33" z="0.12">
         <origin xyz="0 0 0" rpy="0 0 0"/>
       </xacro:inertial_box>
@@ -49,8 +50,59 @@
   </gazebo>
 <!-- LEFT WHEEL FRONT -->
-<joint name="left_wheel_front_joint" type="fixed">
+<xacro:robot_wheel joint_name="left_wheel_front"
+                    joint_type="fixed"
+                    parent="base_link"
+                    origin_x="0.245"
+                    origin_y="0.205"
+                    origin_z="-0.02"
+                    rotation_x="${3*pi/2}"
+                    rotation_y="${pi}"
+                    rotation_z="0"
+                    radius="0.0625"
+                    length="0.08">
+</xacro:robot_wheel>
+<!-- LEFT WHEEL BACK -->
+<xacro:robot_wheel joint_name="left_wheel_back"
+                    joint_type="fixed"
+                    parent="base_link"
+                    origin_x="-0.245"
+                    origin_y="0.205"
+                    origin_z="-0.02"
+                    rotation_x="${3*pi/2}"
+                    rotation_y="${pi}"
+                    rotation_z="0"
+                    radius="0.0625"
+                    length="0.08">
+</xacro:robot_wheel>
+<!-- RIGHT WHEEL FRONT -->
+<xacro:robot_wheel joint_name="right_wheel_front"
+                    joint_type="fixed"
+                    parent="base_link"
+                    origin_x="0.245"
+                    origin_y="-0.205"
+                    origin_z="-0.02"
+                    rotation_x="${pi/2}"
+                    rotation_y="0"
+                    rotation_z="0"
+                    radius="0.0625"
+                    length="0.08">
+</xacro:robot_wheel>
+<!-- RIGHT WHEEL BACK -->
+<xacro:robot_wheel joint_name="right_wheel_back"
+                    joint_type="fixed"
+                    parent="base_link"
+                    origin_x="-0.245"
+                    origin_y="-0.205"
+                    origin_z="-0.02"
+                    rotation_x="${pi/2}"
+                    rotation_y="0"
+                    rotation_z="0"
+                    radius="0.0625"
+                    length="0.08">
+</xacro:robot_wheel>
+<!-- <joint name="left_wheel_front_joint" type="fixed">
   <parent link="base_link"/>
   <child link="left_wheel_front"/>
-  <origin xyz="0.25 0.175 -0.075" rpy="-${pi/2} 0 0"/>
+  <origin xyz="0.245 0.205 -0.02" rpy="-${pi/2} 0 0"/>
   <axis xyz="0 0 1"/>
 </joint>
@@ -59,14 +111,14 @@
     <origin xyz="0 0 0" rpy="0 0 0"/>
       <geometry>
-        <!-- <mesh filename="package://urdf_omni_drive/description/meshes/wheel.STL"/> -->
-        <cylinder radius="0.08" length="0.05"/>
-      </geometry>
-      <material name="black"/>
-  </visual>
-  <collision>
-    <origin xyz="0 0 0" rpy="0 0 0"/>
-      <geometry>
-        <!-- <mesh filename="package://urdf_omni_drive/description/meshes/wheel.STL"/> -->
-        <cylinder radius="0.08" length="0.05"/>
+         <mesh filename="package://urdf_omni_drive/description/meshes/wheel.STL"/>
+        <cylinder radius="0.0625" length="0.08"/>
+      </geometry>
+      <material name="black"/>
+  </visual>
+  <collision>
+    <origin xyz="0 0 0" rpy="0 0 0"/>
+      <geometry>
+        <mesh filename="package://urdf_omni_drive/description/meshes/wheel.STL"/>
+        <cylinder radius="0.0625" length="0.08"/>
       </geometry>
   </collision>
@@ -77,7 +129,6 @@
 <gazebo reference="left_wheel_front">
   <material>Gazebo/DarkGrey</material>
-</gazebo>
-<!-- LEFT WHEEL BACK -->
-<joint name="left_wheel_back_joint" type="fixed">
+</gazebo> -->
+<!-- <joint name="left_wheel_back_joint" type="fixed">
   <parent link="base_link"/>
   <child link="left_wheel_back"/>
@@ -89,13 +140,13 @@
     <origin xyz="0 0 0" rpy="0 0 0"/>
       <geometry>
-        <!-- <mesh filename="package://urdf_omni_drive/description/meshes/wheel.STL"/> -->
-        <cylinder radius="0.08" length="0.05"/>
-      </geometry>
-      <material name="black"/>
-  </visual>
-  <collision>
-    <origin xyz="0 0 0" rpy="0 0 0"/>
-      <geometry>
-        <!-- <mesh filename="package://urdf_omni_drive/description/meshes/wheel.STL"/> -->
+        <mesh filename="package://urdf_omni_drive/description/meshes/wheel.STL"/>
+        <cylinder radius="0.08" length="0.05"/>
+      </geometry>
+      <material name="black"/>
+  </visual>
+  <collision>
+    <origin xyz="0 0 0" rpy="0 0 0"/>
+      <geometry>
+        <mesh filename="package://urdf_omni_drive/description/meshes/wheel.STL"/>
         <cylinder radius="0.08" length="0.05"/>
       </geometry>
@@ -108,5 +159,4 @@
   <material>Gazebo/DarkGrey</material>
 </gazebo>
-<!-- RIGHT WHEEL FRONT -->
 <joint name="right_wheel_front_joint" type="fixed">
   <parent link="base_link"/>
@@ -119,13 +169,13 @@
     <origin xyz="0 0 0" rpy="0 0 0"/>
       <geometry>
-        <!-- <mesh filename="package://urdf_omni_drive/description/meshes/wheel.STL"/> -->
-        <cylinder radius="0.08" length="0.05"/>
-      </geometry>
-      <material name="black"/>
-  </visual>
-  <collision>
-    <origin xyz="0 0 0" rpy="0 0 0"/>
-      <geometry>
-        <!-- <mesh filename="package://urdf_omni_drive/description/meshes/wheel.STL"/> -->
+        <mesh filename="package://urdf_omni_drive/description/meshes/wheel.STL"/>
+        <cylinder radius="0.08" length="0.05"/>
+      </geometry>
+      <material name="black"/>
+  </visual>
+  <collision>
+    <origin xyz="0 0 0" rpy="0 0 0"/>
+      <geometry>
+        <mesh filename="package://urdf_omni_drive/description/meshes/wheel.STL"/>
         <cylinder radius="0.08" length="0.05"/>
       </geometry>
@@ -138,5 +188,4 @@
   <material>Gazebo/DarkGrey</material>
 </gazebo>
-<!-- RIGHT WHEEL BACK -->
 <joint name="right_wheel_back_joint" type="fixed">
   <parent link="base_link"/>
@@ -149,13 +198,13 @@
     <origin xyz="0 0 0" rpy="0 0 0"/>
       <geometry>
-        <!-- <mesh filename="package://urdf_omni_drive/description/meshes/wheel.STL"/> -->
-        <cylinder radius="0.08" length="0.05"/>
-      </geometry>
-      <material name="black"/>
-  </visual>
-  <collision>
-    <origin xyz="0 0 0" rpy="0 0 0"/>
-      <geometry>
-        <!-- <mesh filename="package://urdf_omni_drive/description/meshes/wheel.STL"/> -->
+        <mesh filename="package://urdf_omni_drive/description/meshes/wheel.STL"/>
+        <cylinder radius="0.08" length="0.05"/>
+      </geometry>
+      <material name="black"/>
+  </visual>
+  <collision>
+    <origin xyz="0 0 0" rpy="0 0 0"/>
+      <geometry>
+        <mesh filename="package://urdf_omni_drive/description/meshes/wheel.STL"/>
         <cylinder radius="0.08" length="0.05"/>
       </geometry>
@@ -168,3 +217,4 @@
   <material>Gazebo/DarkGrey</material>
 </gazebo>
+-->
 </robot>
