Commit message: Started implementing lidar and slam

File: description/robot.urdf.xacro (robot description, xacro)
@@ -1,5 +1,6 @@
 <?xml version="1.0"?>
 <robot xmlns:xacro="http://www.ros.org/wiki/xacro"  name="urdf_omni_drive">
-    <xacro:include filename="robot_core.xacro" />
+    <xacro:include filename="robot_core.xacro"/>
+    <xacro:include filename="lidar.xacro"/>
     <xacro:include filename="gazebo_control.xacro"/>
 </robot>

File: description/robot_core.xacro (robot description, xacro)
@@ -9,15 +9,17 @@
     <color rgba="0 0 0 1"/>
 </material>
-<!--
-<link name="base_footprint">
-</link>
-<joint name="odom_joint" type="fixed">
-  <parent link="base_footprint"/>
-  <child link="base_link"/>
-  <origin xyz="0 0 0"/>
-</joint> -->
+<material name="red">
+    <color rgba="0.5 0 0 1"/>
+</material>
 <!-- BASE LINK -->
 <link name="base_link">
 </link>
+<link name="base_footprint">
+</link>
+<joint name="base_footprint_joint" type="fixed">
+  <parent link="base_link"/>
+  <child link="base_footprint"/>
+  <origin xyz="0 0 0"/>
+</joint>
 <!-- CHASSIS -->
 <joint name="chassis_joint" type="fixed">
