Commit message: Xacro changes and updated launch file

File: description/lidar.xacro (robot description, xacro)
@@ -4,5 +4,5 @@
         <parent link="chassis"/>
         <child link="laser_frame"/>
-        <origin xyz="0 0 0.06" rpy="0 0 0"/>
+        <origin xyz="0 0 0.06" rpy="0 0 ${pi}"/>
     </joint>
     <link name="laser_frame">

File: description/robot.urdf.xacro (robot description, xacro)
@@ -3,4 +3,4 @@
     <xacro:include filename="robot_core.xacro"/>
     <xacro:include filename="lidar.xacro"/>
-    <xacro:include filename="gazebo_control.xacro"/>
+    <!-- <xacro:include filename="gazebo_control.xacro"/> -->
 </robot>

File: description/robot_core.xacro (robot description, xacro)
@@ -15,6 +15,4 @@
 <link name="base_link">
 </link>
-<link name="base_footprint">
-</link>
 <joint name="base_footprint_joint" type="fixed">
   <parent link="base_link"/>
@@ -22,4 +20,6 @@
   <origin xyz="0 0 0"/>
 </joint>
+<link name="base_footprint">
+</link>
 <!-- CHASSIS -->
 <joint name="chassis_joint" type="fixed">
