Commit message: Robot moves with omni kinematics, but wheels are static because tf wont work if they are continuous. Need to make separate tf node to publish wheel speeds

File: description/gazebo_control.xacro (robot description, xacro)
@@ -3,10 +3,12 @@
     <gazebo>
         <plugin name="object_controller" filename="libgazebo_ros_planar_move.so">
-            <commandTopic>cmd_vel</commandTopic>
-            <odometryTopic>odom</odometryTopic>
-            <odometryFrame>odom</odometryFrame>
-            <odometryRate>20.0</odometryRate>
-            <robotBaseFrame>chassis</robotBaseFrame>
-          </plugin>
+            <command_topic>cmd_vel</command_topic>
+            <odometry_topic>odom/unfiltered</odometry_topic>
+            <odometry_frame>odom</odometry_frame>
+            <odometry_rate>20.0</odometry_rate>
+            <robot_base_frame>base_link</robot_base_frame>
+            <publish_odom>true</publish_odom>
+            <publish_odom_tf>true</publish_odom_tf>
+        </plugin>
     </gazebo>
 </robot>

File: description/robot_core.xacro (robot description, xacro)
@@ -8,4 +8,12 @@
     <color rgba="0 0 0 1"/>
 </material>
+<!--
+<link name="base_footprint">
+</link>
+<joint name="odom_joint" type="fixed">
+  <parent link="base_footprint"/>
+  <child link="base_link"/>
+  <origin xyz="0 0 0"/>
+</joint> -->
 <!-- BASE LINK -->
 <link name="base_link">
@@ -41,6 +49,6 @@
   </gazebo>
 <!-- LEFT WHEEL FRONT -->
-<joint name="left_wheel_front_joint" type="continuous">
-  <parent link="chassis"/>
+<joint name="left_wheel_front_joint" type="fixed">
+  <parent link="base_link"/>
   <child link="left_wheel_front"/>
   <origin xyz="0.25 0.175 -0.075" rpy="-${pi/2} 0 0"/>
@@ -71,6 +79,6 @@
 </gazebo>
 <!-- LEFT WHEEL BACK -->
-<joint name="left_wheel_back_joint" type="continuous">
-  <parent link="chassis"/>
+<joint name="left_wheel_back_joint" type="fixed">
+  <parent link="base_link"/>
   <child link="left_wheel_back"/>
   <origin xyz="-0.25 0.175 -0.075" rpy="-${pi/2} 0 0"/>
@@ -101,6 +109,6 @@
 </gazebo>
 <!-- RIGHT WHEEL FRONT -->
-<joint name="right_wheel_front_joint" type="continuous">
-  <parent link="chassis"/>
+<joint name="right_wheel_front_joint" type="fixed">
+  <parent link="base_link"/>
   <child link="right_wheel_front"/>
   <origin xyz="0.25 -0.175 -0.075" rpy="${pi/2} 0 0"/>
@@ -131,6 +139,6 @@
 </gazebo>
 <!-- RIGHT WHEEL BACK -->
-<joint name="right_wheel_back_joint" type="continuous">
-  <parent link="chassis"/>
+<joint name="right_wheel_back_joint" type="fixed">
+  <parent link="base_link"/>
   <child link="right_wheel_back"/>
   <origin xyz="-0.25 -0.175 -0.075" rpy="${pi/2} 0 0"/>

Commit message: Wheels now show correctly in Rviz with velocities. For some reason the wheel macro would not work.

File: description/gazebo_control.xacro (robot description, xacro)
@@ -1,5 +1,5 @@
 <?xml version="1.0"?>
 <robot xmlns:xacro="http://www.ros.org/wiki/xacro">
-    <gazebo>
+    <!-- <gazebo>
         <plugin name="object_controller" filename="libgazebo_ros_planar_move.so">
             <command_topic>cmd_vel</command_topic>
@@ -11,4 +11,4 @@
             <publish_odom_tf>true</publish_odom_tf>
         </plugin>
-    </gazebo>
+    </gazebo> -->
 </robot>

File: description/lidar.xacro (robot description, xacro)
@@ -2,5 +2,5 @@
 <robot xmlns:xacro="http://www.ros.org/wiki/xacro">
     <joint name="laser_joint" type="fixed">
-        <parent link="chassis"/>
+        <parent link="base_link"/>
         <child link="laser_frame"/>
         <origin xyz="0 0 0.06" rpy="0 0 ${pi}"/>

File: description/robot_core.xacro (robot description, xacro)
@@ -14,19 +14,4 @@
 <!-- BASE LINK -->
 <link name="base_link">
-</link>
-<joint name="base_footprint_joint" type="fixed">
-  <parent link="base_link"/>
-  <child link="base_footprint"/>
-  <origin xyz="0 0 0"/>
-</joint>
-<link name="base_footprint">
-</link>
-<!-- CHASSIS -->
-<joint name="chassis_joint" type="fixed">
-    <parent link="base_link"/>
-    <child link="chassis"/>
-    <origin xyz="0 0 0"/>
-</joint>
-<link name="chassis">
     <visual>
     <origin xyz="0 0 0" rpy="0 0 0"/>
@@ -48,10 +33,168 @@
       </xacro:inertial_box>
   </link>
+  <gazebo reference="base_link">
+      <material>Gazebo/SkyBlue</material>
+  </gazebo>
+<!-- BASE FOOTPRINT -->
+<link name="base_footprint">
+</link>
+<joint name="base_footprint_joint" type="fixed">
+  <parent link="base_link"/>
+  <child link="base_footprint"/>
+  <origin xyz="0 0 0"/>
+</joint>
+<!--
+ CHASSIS
+<joint name="chassis_joint" type="fixed">
+    <parent link="base_link"/>
+    <child link="chassis"/>
+    <origin xyz="0 0 0"/>
+</joint> -->
+<!-- <link name="chassis">
+    <visual>
+    <origin xyz="0 0 0" rpy="0 0 0"/>
+      <geometry>
+         <mesh filename="package://urdf_omni_drive/description/meshes/frame.STL" scale="0.001 0.001 0.001"/>
+        <box size="0.75 0.33 0.12"/>
+      </geometry>
+      <material name="white"/>
+    </visual>
+    <collision>
+      <origin xyz="0 0 0" rpy="0 0 0"/>
+        <geometry>
+          <mesh filename="package://urdf_omni_drive/description/meshes/frame.STL" scale="0.001 0.001 0.001"/>
+          <box size="0.75 0.33 0.12"/>
+        </geometry>
+      </collision>
+      <xacro:inertial_box mass="5" x="0.75" y="0.33" z="0.12">
+        <origin xyz="0 0 0" rpy="0 0 0"/>
+      </xacro:inertial_box>
+  </link>
   <gazebo reference="chassis">
       <material>Gazebo/SkyBlue</material>
-  </gazebo>
+  </gazebo> -->
 <!-- LEFT WHEEL FRONT -->
-<xacro:robot_wheel joint_name="left_wheel_front"
-                    joint_type="fixed"
+<link name="left_wheel_front">
+  <visual>
+      <origin xyz="0 0 0" rpy="0 0 0"/>
+      <geometry>
+          <!-- <mesh filename="package://urdf_omni_drive/description/meshes/wheel.STL"/> -->
+          <cylinder radius="0.0625" length="0.08"/>
+      </geometry>
+      <material name="black"/>
+  </visual>
+  <collision>
+      <origin xyz="0 0 0" rpy="0 0 0"/>
+      <geometry>
+          <!-- <mesh filename="package://urdf_omni_drive/description/meshes/wheel.STL"/> -->
+          <cylinder radius="0.0625" length="0.08"/>
+      </geometry>
+  </collision>
+  <xacro:inertial_cylinder mass="0.5" radius="0.0625" length="0.08">
+      <origin xyz="0 0 0" rpy="0 0 0"/>
+  </xacro:inertial_cylinder>
+</link>
+<joint name="left_wheel_front" type="continuous">
+  <parent link="base_link"/>
+  <child link="left_wheel_front"/>
+    <origin xyz="0.245 0.205 -0.02" rpy="${3*pi/2} ${pi} 0"/>
+    <axis xyz="0 0 1"/>
+</joint>
+  <gazebo reference="left_wheel_front">
+    <material>Gazebo/DarkGrey</material>
+  </gazebo>
+  <!-- LEFT WHEEL BACK -->
+<link name="left_wheel_back">
+  <visual>
+      <origin xyz="0 0 0" rpy="0 0 0"/>
+      <geometry>
+          <!-- <mesh filename="package://urdf_omni_drive/description/meshes/wheel.STL"/> -->
+          <cylinder radius="0.0625" length="0.08"/>
+      </geometry>
+      <material name="black"/>
+  </visual>
+  <collision>
+      <origin xyz="0 0 0" rpy="0 0 0"/>
+      <geometry>
+          <!-- <mesh filename="package://urdf_omni_drive/description/meshes/wheel.STL"/> -->
+          <cylinder radius="0.0625" length="0.08"/>
+      </geometry>
+  </collision>
+  <xacro:inertial_cylinder mass="0.5" radius="0.0625" length="0.08">
+      <origin xyz="0 0 0" rpy="0 0 0"/>
+  </xacro:inertial_cylinder>
+</link>
+<joint name="left_wheel_back" type="continuous">
+  <parent link="base_link"/>
+  <child link="left_wheel_back"/>
+    <origin xyz="-0.245 0.205 -0.02" rpy="${3*pi/2} ${pi} 0"/>
+    <axis xyz="0 0 1"/>
+</joint>
+  <gazebo reference="left_wheel_back">
+    <material>Gazebo/DarkGrey</material>
+  </gazebo>
+<!-- RIGHT WHEEL FRONT -->
+<link name="right_wheel_front">
+  <visual>
+      <origin xyz="0 0 0" rpy="0 0 0"/>
+      <geometry>
+          <!-- <mesh filename="package://urdf_omni_drive/description/meshes/wheel.STL"/> -->
+          <cylinder radius="0.0625" length="0.08"/>
+      </geometry>
+      <material name="black"/>
+  </visual>
+  <collision>
+      <origin xyz="0 0 0" rpy="0 0 0"/>
+      <geometry>
+          <!-- <mesh filename="package://urdf_omni_drive/description/meshes/wheel.STL"/> -->
+          <cylinder radius="0.0625" length="0.08"/>
+      </geometry>
+  </collision>
+  <xacro:inertial_cylinder mass="0.5" radius="0.0625" length="0.08">
+      <origin xyz="0 0 0" rpy="0 0 0"/>
+  </xacro:inertial_cylinder>
+</link>
+<joint name="right_wheel_front" type="continuous">
+  <parent link="base_link"/>
+  <child link="right_wheel_front"/>
+    <origin xyz="0.245 -0.205 -0.02" rpy="${pi/2} 0 0"/>
+    <axis xyz="0 0 1"/>
+</joint>
+  <gazebo reference="right_wheel_front">
+    <material>Gazebo/DarkGrey</material>
+  </gazebo>
+<!-- RIGHT WHEEL BACK -->
+<link name="right_wheel_back">
+  <visual>
+      <origin xyz="0 0 0" rpy="0 0 0"/>
+      <geometry>
+          <!-- <mesh filename="package://urdf_omni_drive/description/meshes/wheel.STL"/> -->
+          <cylinder radius="0.0625" length="0.08"/>
+      </geometry>
+      <material name="black"/>
+  </visual>
+  <collision>
+      <origin xyz="0 0 0" rpy="0 0 0"/>
+      <geometry>
+          <!-- <mesh filename="package://urdf_omni_drive/description/meshes/wheel.STL"/> -->
+          <cylinder radius="0.0625" length="0.08"/>
+      </geometry>
+  </collision>
+  <xacro:inertial_cylinder mass="0.5" radius="0.0625" length="0.08">
+      <origin xyz="0 0 0" rpy="0 0 0"/>
+  </xacro:inertial_cylinder>
+</link>
+<joint name="right_wheel_back" type="continuous">
+  <parent link="base_link"/>
+  <child link="right_wheel_back"/>
+    <origin xyz="-0.245 -0.205 -0.02" rpy="${3*pi/2} ${pi} 0"/>
+    <axis xyz="0 0 1"/>
+</joint>
+  <gazebo reference="right_wheel_back">
+    <material>Gazebo/DarkGrey</material>
+  </gazebo>
+<!-- LEFT WHEEL FRONT -->
+<!-- <xacro:robot_wheel joint_name="left_wheel_front"
+                    joint_type="continuous"
                     parent="base_link"
                     origin_x="0.245"
@@ -63,8 +206,8 @@
                     radius="0.0625"
                     length="0.08">
-</xacro:robot_wheel>
+</xacro:robot_wheel> -->
 <!-- LEFT WHEEL BACK -->
-<xacro:robot_wheel joint_name="left_wheel_back"
-                    joint_type="fixed"
+<!-- <xacro:robot_wheel joint_name="left_wheel_back"
+                    joint_type="continuous"
                     parent="base_link"
                     origin_x="-0.245"
@@ -76,8 +219,8 @@
                     radius="0.0625"
                     length="0.08">
-</xacro:robot_wheel>
+</xacro:robot_wheel> -->
 <!-- RIGHT WHEEL FRONT -->
-<xacro:robot_wheel joint_name="right_wheel_front"
-                    joint_type="fixed"
+<!-- <xacro:robot_wheel joint_name="right_wheel_front"
+                    joint_type="continuous"
                     parent="base_link"
                     origin_x="0.245"
@@ -89,8 +232,8 @@
                     radius="0.0625"
                     length="0.08">
-</xacro:robot_wheel>
+</xacro:robot_wheel> -->
 <!-- RIGHT WHEEL BACK -->
-<xacro:robot_wheel joint_name="right_wheel_back"
-                    joint_type="fixed"
+<!-- <xacro:robot_wheel joint_name="right_wheel_back"
+                    joint_type="continuous"
                     parent="base_link"
                     origin_x="-0.245"
@@ -102,5 +245,5 @@
                     radius="0.0625"
                     length="0.08">
-</xacro:robot_wheel>
+</xacro:robot_wheel> -->
 <!-- <joint name="left_wheel_front_joint" type="fixed">
   <parent link="base_link"/>

File: description/robot_macros.xacro (robot description, xacro)
@@ -2,10 +2,4 @@
 <robot xmlns:xacro="http://www.ros.org/wiki/xacro" >
 <xacro:macro name="robot_wheel" params="joint_name joint_type parent origin_x origin_y origin_z rotation_x rotation_y rotation_z radius length">
-    <joint name="${joint_name}_joint" type="${joint_type}">
-    <parent link="${parent}"/>
-    <child link="${joint_name}"/>
-    <origin xyz="${origin_x} ${origin_y} ${origin_z}" rpy="${rotation_x} ${rotation_y} ${rotation_z}"/>
-    <axis xyz="0 0 1"/>
-    </joint>
     <link name="${joint_name}">
     <visual>
@@ -28,4 +22,10 @@
     </xacro:inertial_cylinder>
     </link>
+    <joint name="${joint_name}_joint" type="${joint_type}">
+    <parent link="${parent}"/>
+    <child link="${joint_name}"/>
+    <origin xyz="${origin_x} ${origin_y} ${origin_z}" rpy="${rotation_x} ${rotation_y} ${rotation_z}"/>
+    <axis xyz="0 0 1"/>
+    </joint>
     <gazebo reference="${joint_name}">
     <material>Gazebo/DarkGrey</material>
